Commit message: update architecture;

File: resources/z1/z1.urdf (robot description, URDF)
Before this commit: robot z1, 9 links, 8 joints
Links:
- added link gripperMover, mass 0.27621302; collision mesh filename=meshes/collision/z1_GripperMover.obj scale=1 1 1; visual mesh filename=meshes/visual/z1_GripperMover.dae scale=1 1 1
- added link gripperStator, mass 0.52603655; collision mesh filename=meshes/collision/z1_GripperStator.obj scale=1 1 1; visual mesh filename=meshes/visual/z1_GripperStator.dae scale=1 1 1
Joints:
- added joint gripperStator: type fixed, parent link06, child gripperStator, origin xyz=0.051 0.0 0.0 rpy=0 0 0
- added joint jointGripper: type fixed, parent gripperStator, child gripperMover, origin xyz=0.049 0.0 0 rpy=0 0 0, axis 0 1 0, limit lower=-1.5707963267948966 upper=0.0 effort=30.0 velocity=3.1415
- joint endEffector: parent link06 -> gripperStator
